Commit message: Add lidar sensor, human model and Gazebo sensors world
- Add safety lidar (gpu_lidar, 360 rays, 10m range, gaussian noise) mounted on link1 at 1.2m height
- Add custom Gazebo world with gz::sim::systems::Sensors plugin (required for sensor data)
- Add human_dummy SDF model (cylinder 0.5m diameter, 1.75m height) for safety testing
- Bridge /scan topic from Gazebo to ROS2 via ros_gz_bridge
- Add move_group_sim.launch.py with explicit use_sim_time (fixes MoveIt2 execution with Gazebo)
- Fix safety_monitor_node: use control_msgs/SpeedScalingFactor with matching QoS profile

File: puma560_description/urdf/puma560_robot.urdf.xacro (robot description, xacro)
@@ -14,4 +14,7 @@
   <material name="green">
     <color rgba="0 0.8 0 0.8"/>
+  </material>
+  <material name="black">
+    <color rgba="0.1 0.1 0.1 1"/>
   </material>
   <xacro:property name="M_PI" value="3.14159265"/>
@@ -55,4 +58,28 @@
     </inertial>
   </link>
+  <!-- ===== Lidar sensor (safety scanner), stationary on robot base ===== -->
+  <link name="lidar_link">
+    <visual>
+      <geometry>
+        <cylinder radius="0.05" length="0.07"/>
+      </geometry>
+      <material name="black"/>
+    </visual>
+    <collision>
+      <geometry>
+        <cylinder radius="0.05" length="0.07"/>
+      </geometry>
+    </collision>
+    <inertial>
+      <origin xyz="0 0 0" rpy="0 0 0"/>
+      <mass value="0.2"/>
+      <inertia ixx="0.0001" ixy="0" ixz="0" iyy="0.0001" iyz="0" izz="0.0001"/>
+    </inertial>
+  </link>
+  <joint name="link1_to_lidar" type="fixed">
+    <parent link="link1"/>
+    <child link="lidar_link"/>
+    <origin xyz="0 0 1.2" rpy="0 0 0"/>
+  </joint>
   <link name="link2">
     <visual>
@@ -355,3 +382,39 @@
     <mu2>1.0</mu2>
   </gazebo>
+  <!-- ===== Gazebo lidar sensor ===== -->
+  <gazebo reference="lidar_link">
+    <sensor name="safety_lidar" type="gpu_lidar">
+      <pose>0 0 0 0 0 0</pose>
+      <topic>scan</topic>
+      <update_rate>10</update_rate>
+      <always_on>true</always_on>
+      <visualize>true</visualize>
+      <lidar>
+        <scan>
+          <horizontal>
+            <samples>360</samples>
+            <resolution>1</resolution>
+            <min_angle>-3.14159</min_angle>
+            <max_angle>3.14159</max_angle>
+          </horizontal>
+          <vertical>
+            <samples>1</samples>
+            <resolution>1</resolution>
+            <min_angle>0</min_angle>
+            <max_angle>0</max_angle>
+          </vertical>
+        </scan>
+        <range>
+          <min>0.1</min>
+          <max>10.0</max>
+          <resolution>0.01</resolution>
+        </range>
+        <noise>
+          <type>gaussian</type>
+          <mean>0.0</mean>
+          <stddev>0.01</stddev>
+        </noise>
+      </lidar>
+    </sensor>
+  </gazebo>
 </robot>

Commit message: Add lidar-based human detection and unified system launch
- Add lidar_human_detector: clustering of laser scan data, object position
  estimation in world frame (~4cm accuracy), RViz marker publishing
- Filter out robot's own links from detection using TF lookup
  (fixes false STOP when arm enters scan plane)
- Merge split clusters caused by beam gaps on cylindrical objects
- Select largest cluster instead of nearest one
- Move lidar from 1.2m to 0.5m height (avoids arm workspace)
- Fix distance calculation in safety_monitor: subtract object radius,
  use horizontal projection for vertically extended objects
- Add full_system.launch.py: single command starts Gazebo, robot,
  human model, detector, safety monitor and preconfigured RViz
- Add RViz config with robot model, safety zones, detection markers
  and raw laser scan visualization

File: puma560_description/urdf/puma560_robot.urdf.xacro (robot description, xacro)
@@ -80,5 +80,5 @@
     <parent link="link1"/>
     <child link="lidar_link"/>
-    <origin xyz="0 0 1.2" rpy="0 0 0"/>
+    <origin xyz="0 0 0.5" rpy="0 0 0"/>
   </joint>
   <link name="link2">

Commit message: Add depth camera detection and multi-sensor fusion
- Add RGB-D camera to URDF (320x240, 10Hz, mounted 2.5m above and 1.5m
  behind robot base, tilted 43 deg down) with gaussian depth noise
- Bridge camera topics (image, depth_image, points, camera_info) to ROS2
- Add camera_human_detector: OpenCV-based detection on depth image
  (inRange threshold, morphological filtering, contour extraction,
  pinhole projection to 3D), ~3cm position accuracy
- Filter floor and ceiling by computing per-pixel height in world frame
- Reject detections overlapping robot links via TF lookup
- Publish debug mask image with contours for visualization
- Add sensor_fusion_node: weighted combination of lidar and camera
  estimates with freshness timeout, automatic fallback to single sensor
  on occlusion, disagreement handling
- Rename lidar detector output to /puma/human_position_lidar
- Wrap robot_description in ParameterValue (fixes YAML parsing error)
- Compensate object radius in camera depth estimate
- Extend full_system.launch.py with camera detector and fusion nodes

File: puma560_description/urdf/puma560_robot.urdf.xacro (robot description, xacro)
@@ -82,4 +82,36 @@
     <origin xyz="0 0 0.5" rpy="0 0 0"/>
   </joint>
+  <!-- ===== Depth camera (overhead workspace monitoring) ===== -->
+  <link name="camera_link">
+    <visual>
+      <geometry>
+        <box size="0.08 0.12 0.05"/>
+      </geometry>
+      <material name="black"/>
+    </visual>
+    <collision>
+      <geometry>
+        <box size="0.08 0.12 0.05"/>
+      </geometry>
+    </collision>
+    <inertial>
+      <origin xyz="0 0 0" rpy="0 0 0"/>
+      <mass value="0.3"/>
+      <inertia ixx="0.0002" ixy="0" ixz="0" iyy="0.0002" iyz="0" izz="0.0002"/>
+    </inertial>
+  </link>
+  <!-- Камера смещена назад и вверх, наклонена вниз на 35 градусов -->
+  <joint name="link1_to_camera" type="fixed">
+    <parent link="link1"/>
+    <child link="camera_link"/>
+    <origin xyz="-1.5 0 2.5" rpy="0 0.75 0"/>
+  </joint>
+  <!-- Оптический кадр: ROS-конвенция (z вперёд, x вправо, y вниз) -->
+  <link name="camera_optical_frame"/>
+  <joint name="camera_to_optical" type="fixed">
+    <parent link="camera_link"/>
+    <child link="camera_optical_frame"/>
+    <origin xyz="0 0 0" rpy="${-M_PI/2} 0 ${-M_PI/2}"/>
+  </joint>
   <link name="link2">
     <visual>
@@ -418,3 +450,36 @@
     </sensor>
   </gazebo>
+  <!-- ===== Gazebo depth camera sensor ===== -->
+  <gazebo reference="camera_link">
+    <sensor name="workspace_camera" type="rgbd_camera">
+      <topic>camera</topic>
+      <update_rate>10</update_rate>
+      <always_on>true</always_on>
+      <visualize>true</visualize>
+      <gz_frame_id>camera_optical_frame</gz_frame_id>
+      <camera>
+        <horizontal_fov>1.204</horizontal_fov>
+        <image>
+          <width>320</width>
+          <height>240</height>
+          <format>R8G8B8</format>
+        </image>
+        <clip>
+          <near>0.3</near>
+          <far>8.0</far>
+        </clip>
+        <depth_camera>
+          <clip>
+            <near>0.3</near>
+            <far>8.0</far>
+          </clip>
+        </depth_camera>
+        <noise>
+          <type>gaussian</type>
+          <mean>0.0</mean>
+          <stddev>0.007</stddev>
+        </noise>
+      </camera>
+    </sensor>
+  </gazebo>
 </robot>
